File: pickit2_smd.sch (KiCad schematic (older format))
At the start: 54 parts, among them CON1 USB-MINI-B, P1 CONN_6, Q1 MOSFET_P, Q2 MOSFET_N, Q3 MOSFET_P, Q4 MOSFET_N, Q5 MOSFET_N, Q6 MOSFET_P, Q7 MOSFET_N, Q8 20MHz, SW1 SW_PUSH_SMALL, U1 LM358, U2 PIC18F2550

Commit message: versao modificada, PCB 50%
Parts:
- added C13: 100n, symbol C
- added D6: DIODE, symbol DIODE
- added Q10, Q11, Q9: PNP, symbol PNP
- added R24, R25, R26, R30: 33, symbol R
- added R27: 820, symbol R
- added R28, R29, R32, R33, R34, R35: R, symbol R
- added R31: 10k, symbol R
- added R36: 0, symbol R
- added unit 2 of U1
- added U3, U4: 24C512, symbol 24C512
- D3: value DIODE -> bat54
Connections:
- net +5V: now also R28.1, R31.1, R32.1, R34.1, R35.1, U3.8 (VCC), U4.8 (VCC)
- net GND: now also C13.2, Q10.3 (C), Q11.3 (C), Q9.3 (C), R27.1, R29.2, R33.2, U1.5 (+), U1.6 (-), U3.1 (A0), U3.3 (A2), U3.4 (GND), U4.1 (A0), U4.3 (A2), U4.4 (GND)
- net RA2: now also R24.1; no longer R16.1
- net RA3: now also R25.1; no longer R17.1
- net RA4: now also R26.1; no longer R20.1
- net RB0: now also R35.2, U3.5 (SDA), U4.5 (SDA)
- net RB1: now also R34.2, U3.6 (SCL), U4.6 (SCL)
- net RB2: now also R36.1, R36.2
- net RB5: now also R30.1; no longer SW1.1
- net RC6: now also U3.7 (WP), U4.7 (WP)
- net at D5.2 (K), P1.2, R13.1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: now also D6.1 (A)
- new net: Q9.1 (E), R16.1, R24.2
- new net: Q10.1 (E), R17.1, R25.2
- new net: Q11.1 (E), R20.1, R26.2
- new net: C13.1, R30.2, R31.2, SW1.1
- new net: R28.2, R29.1, U3.2 (A1)
- new net: R32.2, R33.1, U4.2 (A1)
- new net clamp: D6.2 (K), Q10.2 (B), Q11.2 (B), Q9.2 (B), R27.2
Other:
- moved on the sheet: R20

Commit message: placa feita
Parts:
- removed C7: CAPAPOL, symbol CAPAPOL
- added C7: 470n, symbol C
- added R37, R38, R39, R40, R41, R42: 0, symbol R
- renumbered C5 to C4, C4 to C5
Connections:
- net GND: now also CON1.6 (SHELL1), CON1.7 (SHELL2), CON1.8 (SHELL3), CON1.9 (SHELL4), C7.2, R37.1, R37.2, R38.1, R38.2, R39.1, R39.2, R40.1, R40.2, R42.1, R42.2
- net at U2.14 (Vusb): now also C7.1
- net at C3.1, C5.1, Q1.D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: now also R41.1; no longer C4.1, L1.2, Q3.S
- new net: C4.1, L1.2, Q3.S, R41.2

Commit message: feito, shunt
Parts:
- added R43: 10K, symbol R
Connections:
- net +5V: now also R43.2
- net RB4: now also R43.1
Changed lines of the file:
@@
 LIBS:transistors_gaui
 LIBS:pickit2_smd-cache
-EELAYER 24 0
+EELAYER 27 0
 EELAYER END
 $Descr A4 11693 8268
@@
 Sheet 1 1
 Title ""
-Date ""
+Date "18 mar 2014"
 Rev ""
 Comp ""
@@
 	1    0    0    -1
 $EndComp
+$Comp
+L R R43
+U 1 1 5328DF4E
+P 3650 2250
+F 0 "R43" V 3730 2250 40  0000 C CNN
+F 1 "10K" V 3657 2251 40  0000 C CNN
+F 2 "" V 3580 2250 30  0000 C CNN
+F 3 "" H 3650 2250 30  0000 C CNN
+	1    3650 2250
+	0    1    1    0
+$EndComp
+Wire Wire Line
+	3900 2250 3900 2300
+Connection ~ 3900 2300
+$Comp
+L +5V #PWR051
+U 1 1 5328DFF9
+P 3400 2250
+F 0 "#PWR051" H 3400 2340 20  0001 C CNN
+F 1 "+5V" H 3400 2340 30  0000 C CNN
+F 2 "" H 3400 2250 60  0000 C CNN
+F 3 "" H 3400 2250 60  0000 C CNN
+	1    3400 2250
+	1    0    0    -1
+$EndComp
